Commit message: doing more work

File: go2_description/urdf/go2_BACKUP.urdf (robot description, URDF)
Before this commit: robot go2_description, 42 links, 41 joints
Links:
- link FL_calflower: mass 0.001 -> None
- link FL_calflower1: mass 0.001 -> None
- link FR_calflower: mass 0.001 -> None
- link FR_calflower1: mass 0.001 -> None
- link RL_calflower: mass 0.001 -> None
- link RL_calflower1: mass 0.001 -> None
- link RR_calflower: mass 0.001 -> None
- link RR_calflower1: mass 0.001 -> None
- link front_camera: mass 0.001 -> None
